File: doc/digispark_adns2620.sch (EAGLE design)
At the start: 30 parts, among them IC1 ATTINY85, IC2 ADNS-2620/2610, Q1 24 MhZ, Q7 2N3906, X1 USBPCB

Commit message: added adjustment of the laser power
Parts:
- removed Q7: 2N3906, transistor-small-signal:2N3906
- removed R22: 100k, rcl:R-EU_R0805
- added C2_3: 10µ, rcl:C-EUC0805K
- added D4: MBR0520LT, diode:MBR0520LT
- LED1: value HLMP-ED80- -> Laser module
- R23: value 47R -> 91R
- R34: value 1k -> 68R
Connections:
- removed net N$168: IC2.LED_CNTL, R34.2
- removed net N$169: Q7.B, R22.1, R34.1
- removed net N$171: LED1.A, R23.1
- removed net N$172: LED1.C, Q7.E
- new net N$13: LED1.C, R23.2
- new net N$24: C2_3.1, LED1.A, R34.1
- new net N$25: D4.C, R34.2
- new net N$26: D4.A, JP5.1
- net 5V: now also D3.C; no longer D3.A
- net GND: now also C2_3.2, R23.1; no longer Q7.C
- net N$16: now also D3.A; no longer D3.C
- net VDD: no longer R22.2, R23.2
Other:
- moved on the sheet: D3, R34
